File: Mainboard/MBC-1000_Mainboard/MBC-1000_Mainboard.kicad_sch (KiCad schematic)
At the start: 6 parts, among them U1 Z80CPU

Commit message: Start mainboard RAM schematic
Parts:
- added A3, D10: 74LS10, symbol 74xx:74LS10
- added B3, C8, F10: 74LS02, symbol 74xx:74LS02
- added B4: 74128, symbol 74xx_IEEE:74128
- added B5, D5: 74LS245, symbol 74xx:74LS245
- added B6: 74LS138, symbol 74xx:74LS138
- added B7, B8, D4, D7: 74LS244, symbol 74xx:74LS244
- added B9: 2716, symbol MBC-1000_Mainboard:2716
- added C12, C13, D12, D13, E12, E13, F12, F13: 4164, symbol MBC-1000_Mainboard:4164
- added C3, E4: 74LS161, symbol 74xx:74LS161
- added C4, C6, E10, F11: 74LS00, symbol 74xx:74LS00
- added C5, E11, G4: 74LS04, symbol 74xx:74LS04
- added C7: 74LS107, symbol 74xx:74LS107
- added C9, D11, G12, U2: 74LS32, symbol 74xx:74LS32
- added D6, D8, E6, E8, F7, F9: 74LS157, symbol 74xx:74LS157
- added D9: MC68B45, Package_DIP:DIP-40_W15.24mm, symbol GPU:MC68B45
- added E5: 74LS30, symbol 74xx:74LS30
- added E7: 74LS374, symbol 74xx:74LS374
- added F4: MB8876A, symbol MBC-1000_Mainboard:MB8876A
- added F6, F8: 2116, symbol MBC-1000_Mainboard:2116
- added G10: MC14585, symbol MBC-1000_Mainboard:MC14585
- added G11, G9: 74LS74, symbol 74xx:74LS74
Connections:
- net GND: now also C10.15 (E), C10.8 (GND), C11.15 (E), C11.8 (GND), C12.16 (Vss), C13.16 (Vss), D12.16 (Vss), D13.16 (Vss), E12.16 (Vss), E13.16 (Vss), F12.16 (Vss), F13.16 (Vss)
- net BUS-A1: now reaches C10.10 (I1c)
- net BUS-A1: now also B1.11 (O5b)
- net BUS-A8: now reaches C10.11 (I0c)
- net BUS-A8: now also A1.5 (O2a)
- net MEM-A3: now reaches C10.12 (Zd)
- net MEM-A3: now also C12.12 (A3), C13.12 (A3), D12.12 (A3), D13.12 (A3), E12.12 (A3), E13.12 (A3), F12.12 (A3), F13.12 (A3)
- net BUS-A10: now reaches C10.13 (I1d)
- net BUS-A10: now also A1.3 (O1a)
- net BUS-A3: now reaches C10.14 (I0d)
- net BUS-A3: now also B1.13 (O6b)
- net VCC: now reaches C10.16 (VCC)
- net VCC: now also A1.16 (VCC), A2.16 (VCC), B1.16 (VCC), C11.16 (VCC), C12.8 (Vcc), C13.8 (Vcc), D12.8 (Vcc), D13.8 (Vcc), E12.8 (Vcc), E13.8 (Vcc), F12.8 (Vcc), F13.8 (Vcc), G9.10 (~{S2}), G9.12 (D2), G9.14 (VCC)
- net BUS-A7: now reaches C10.2 (I0a)
- net BUS-A7: now also A1.11 (O5b)
- net BUS-A0: now reaches C10.3 (I1a)
- net BUS-A0: now also B1.7 (O3a)
- net MEM-A0: now reaches C10.4 (Za)
- net MEM-A0: now also C12.5 (A0), C13.5 (A0), D12.5 (A0), D13.5 (A0), E12.5 (A0), E13.5 (A0), F12.5 (A0), F13.5 (A0)
- net BUS-A9: now reaches C10.5 (I0b)
- net BUS-A9: now also A1.13 (O6b)
- net BUS-A2: now reaches C10.6 (I1b)
- net BUS-A2: now also B1.5 (O2a)
- net MEM-A2: now reaches C10.7 (Zb)
- net MEM-A2: now also C12.6 (A2), C13.6 (A2), D12.6 (A2), D13.6 (A2), E12.6 (A2), E13.6 (A2), F12.6 (A2), F13.6 (A2)
- net MEM-A1: now reaches C10.9 (Zc)
- net MEM-A1: now also C12.7 (A1), C13.7 (A1), D12.7 (A1), D13.7 (A1), E12.7 (A1), E13.7 (A1), F12.7 (A1), F13.7 (A1)
- net BUS-A14: now reaches A2.11 (O5b)
- net BUS-A14: now also C11.10 (I1c)
- net BUS-A12: now reaches A2.13 (O6b)
- net BUS-A12: now also C11.5 (I0b)
- net BUS-A11: now reaches A2.3 (O1a)
- net BUS-A11: now also C11.13 (I1d)
- net BUS-A13: now reaches A2.5 (O2a)
- net BUS-A13: now also C11.2 (I0a)
- net BUS-A15: now reaches A2.7 (O3a)
- net BUS-A15: now also C11.11 (I0c)
- net MEM-A4: now reaches C11.12 (Zd)
- net MEM-A4: now also C12.11 (A4), C13.11 (A4), D12.11 (A4), D13.11 (A4), E12.11 (A4), E13.11 (A4), F12.11 (A4), F13.11 (A4)
- net BUS-A4: now reaches C11.14 (I0d)
- net BUS-A4: now also B1.3 (O1a)
- net BUS-A6: now reaches C11.3 (I1a)
- net BUS-A6: now also A1.7 (O3a)
- net MEM-A6: now reaches C11.4 (Za)
- net MEM-A6: now also C12.13 (A6), C13.13 (A6), D12.13 (A6), D13.13 (A6), E12.13 (A6), E13.13 (A6), F12.13 (A6), F13.13 (A6)
- net BUS-A5: now reaches C11.6 (I1b)
- net BUS-A5: now also A1.9 (O4a)
- net MEM-A5: now reaches C11.7 (Zb)
- net MEM-A5: now also C12.10 (A5), C13.10 (A5), D12.10 (A5), D13.10 (A5), E12.10 (A5), E13.10 (A5), F12.10 (A5), F13.10 (A5)
- net MEM-A7: now reaches C11.9 (Zc)
- net MEM-A7: now also C12.9 (A7), C13.9 (A7), D12.9 (A7), D13.9 (A7), E12.9 (A7), E13.9 (A7), F12.9 (A7), F13.9 (A7)
- net CPU-D6: now reaches U1.10 (D6)
- net CPU-D6: now also F12.14 (DO), F12.2 (DI)
- net CPU-D2: now reaches U1.11 (VCC)
- net CPU-D2: now also D12.14 (DO), D12.2 (DI)
- net CPU-D7: now reaches U1.13 (D7)
- net CPU-D7: now also F13.14 (DO), F13.2 (DI)
- net CPU-D0: now reaches U1.14 (D0)
- net CPU-D0: now also C12.14 (DO), C12.2 (DI)
- net CPU-D1: now reaches U1.15 (D1)
- net CPU-D1: now also C13.14 (DO), C13.2 (DI)
- net ~{CPU-MREQ}: now reaches U1.19 (~{MREQ})
- net ~{CPU-MREQ}: now also B9.20 (~{OE}), E11.1 (A1), F10.3 (B1)
- net ~{CPU-WR}: now reaches U1.22 (~{WR})
- net ~{CPU-WR}: now also B1.10 (I4)
- net ~{CPU-RFSH}: now reaches U1.28 (~{RFSH})
- net ~{CPU-RFSH}: now also D10.11 (3C), D10.13 (1C), G9.11 (C2)
- net CPU-D4: now reaches U1.7 (D4)
- net CPU-D4: now also E12.14 (DO), E12.2 (DI)
- net CPU-D3: now reaches U1.8 (D3)
- net CPU-D3: now also D13.14 (DO), D13.2 (DI)
- net CPU-D5: now reaches U1.9 (D5)
- net CPU-D5: now also E13.14 (DO), E13.2 (DI)
- net ~{BUS-WR}: now reaches B1.9 (O4a)
- net ~{BUS-WR}: now also C12.3 (~{WE}), C13.3 (~{WE}), D12.3 (~{WE}), D13.3 (~{WE}), E12.3 (~{WE}), E13.3 (~{WE}), F12.3 (~{WE}), F13.3 (~{WE})
- new net: E11.10 (Y5), F10.2 (A1)
- new net: E11.11 (A5), E11.12 (Y6)
- new net: D10.8 (3Y), E11.13 (A6)
- new net: D10.9 (3A), D11.8 (Y3)
- new net BUS-MREQ: E11.2 (Y1)
- new net MEM-CAS: E11.9 (A4), F10.1 (Y1)
- new net MEM-RAS: D10.10 (3B), E11.4 (Y2)
- new net ~{MEM-CAS}: C12.15 (~{CAS}), C13.15 (~{CAS}), D12.15 (~{CAS}), D13.15 (~{CAS}), E11.8 (Y4), E12.15 (~{CAS}), E13.15 (~{CAS}), F12.15 (~{CAS}), F13.15 (~{CAS})
- new net ~{MEM-RAS}: C12.4 (~{RAS}), C13.4 (~{RAS}), D12.4 (~{RAS}), D13.4 (~{RAS}), E10.11 (Y4), E11.3 (A2), E12.4 (~{RAS}), E13.4 (~{RAS}), F12.4 (~{RAS}), F13.4 (~{RAS})

Commit message: Continue mainboard logic schematic
Parts:
- added G3: 16M, Oscillator:Oscillator_DIP-14, symbol Oscillator:ACO-xxxMHz-A
- added J1: Keyboard, symbol Connector_Generic:Conn_02x08_Row_Letter_First
- added JP1: Jumper_2_Open, symbol Jumper:Jumper_2_Open
- added R33, R34, R36: 3k3, symbol Device:R_Small_US
- added R35, R37: 100k, symbol Device:R_Small_US
- added R41: 220R, symbol Device:R_Small_US
Connections:
- net BUS-A0: now also B7.15 (I2b), B9.8 (A0)
- net BUS-A1: now also B7.17 (I3b), B9.7 (A1), E11.5 (A3), G12.1 (A1)
- net BUS-A10: now also B9.19 (A10)
- net BUS-A2: now also B6.1 (A0), B7.2 (I0a), B9.6 (A2)
- net BUS-A3: now also B6.2 (A1), B7.4 (I1a), B9.5 (A3)
- net BUS-A4: now also B6.3 (A2), B7.6 (I2a), B9.4 (A4)
- net BUS-A5: now also B7.8 (I3a), B9.3 (A5), D10.3 (2A)
- net BUS-A6: now also B8.11 (I0b), B9.2 (A6), D10.5 (2C)
- net BUS-A7: now also B8.13 (I1b), B9.1 (A7), D10.4 (2B)
- net BUS-A8: now also B9.23 (A8)
- net BUS-A9: now also B9.22 (A9)
- net CPU-D0: now also B9.9 (Q0)
- net CPU-D1: now also B9.10 (Q1)
- net CPU-D2: now also B9.11 (Q2), U1.12 (D2); no longer U1.11 (VCC)
- net CPU-D3: now also B9.13 (Q3)
- net CPU-D4: now also B9.14 (Q4)
- net CPU-D5: now also B9.15 (Q5)
- net CPU-D6: now also B9.16 (Q6)
- net CPU-D7: now also B9.17 (Q7)
- net GND: now also B6.5 (E2), B6.8 (GND), B7.1 (OEa), B7.10 (GND), B7.19 (OEb), B8.1 (OEa), B8.10 (GND), B8.19 (OEb), B9.12 (GND), C6.7 (GND), C7.7 (GND), C8.7 (GND), C9.7 (GND), D10.7 (GND), D11.7 (GND), E10.7 (GND), E11.7 (GND), F10.7 (GND), F11.7 (GND), F9.8 (GND), G10.8 (Vss), G11.7 (GND), G12.7 (GND), G9.7 (GND), U1.29 (GND)
- net VCC: now also B6.16 (VCC), B6.6 (E3), B7.20 (VCC), B8.20 (VCC), B9.21 (Vpp), B9.24 (Vcc), C6.14 (VCC), C7.14 (VCC), C8.14 (VCC), C9.14 (VCC), D10.14 (VCC), D11.14 (VCC), E10.14 (VCC), F10.14 (VCC), F11.14 (VCC), G10.16 (Vdd), G11.12 (D2), G11.14 (VCC), G12.14 (VCC), U1.11 (VCC), R33.2, R34.2, R36.1, R37.2, R41.2
- net ~{CPU-RFSH}: now also B8.15 (I2b)
- net ~{CPU-WR}: now also B7.11 (I0b), C9.1 (A1), D10.1 (1A)
- net ~{BUS-IORD}: now reaches C9.11 (Y4)
- net ~{BUS-IORD}: now also C8.9 (B3)
- net ~{CPU-RD}: now reaches C9.12 (A4)
- net ~{CPU-RD}: now also B7.13 (I1b), D10.2 (1B), U1.21 (~{RD})
- net ~{CPU-IORQ}: now reaches C9.13 (B4)
- net ~{CPU-IORQ}: now also B8.6 (I2a), C9.2 (B1), U1.20 (~{IORQ})
- net ~{BUS-IOWR}: now reaches C9.3 (Y1)
- net ~{BUS-IOWR}: now also C7.12 (C1), F11.2 (B1), G12.10 (B3)
- net IO-CE: now reaches C9.5 (B2)
- net IO-CE: now also C8.10 (Y3)
- net ~{BUS-A6}: now reaches C9.9 (A3)
- net at B6.10 (O5): now also C6.13 (B4)
- net at B6.11 (O4): now also C6.12 (A4)
- net ~{CRTC-CE}: now reaches B6.12 (O3)
- net ~{CRTC-CE}: now also D9.25 (~{CS})
- net ~{PPI-CE}: now reaches B6.13 (O2)
- net ~{FDC-CE}: now reaches B6.14 (O1)
- net ~{FDC-CE}: now also F4.3 (~{CS})
- net at B6.15 (O0): now also G12.9 (A3)
- net ~{IO-CE}: now reaches B6.4 (E1)
- net ~{IO-CE}: now also C8.11 (A4), C8.12 (B4), D10.6 (2Y)
- net at B6.7 (O7): now also C6.1 (A1)
- net at B6.9 (O6): now also C6.2 (B1)
- net at E8.1 (S): now also C6.8 (Y3), D8.1 (S), F9.1 (S)
- net at C8.13 (Y4): now also C8.8 (A3)
- net ~{CPU-RST}: now reaches F11.10 (B3)
- net ~{CPU-RST}: now also E10.5 (B2), G10.15 (A3), U1.26 (~{RESET})
- net at F11.9 (A3): now also G12.3 (Y1)
- net at B8.17 (I3b): now also A2.10 (I4), E4.13 (Q1), E5.4 (D1)
- net ~{CPU-M1}: now reaches B8.8 (I3a)
- net ~{CPU-M1}: now also F10.12 (B4), U1.27 (~{M1})
- net at F7.1 (S): now also C6.6 (Y2), D6.1 (S), E6.1 (S)
- net at F10.11 (A4): now also A2.9 (O4a)
- net at F10.13 (Y4): now also E10.9 (A3)
- net at F10.5 (A2): now also G10.4 (A>B)
- net at F10.6 (B2): now also G10.2 (A2)
- net at E11.6 (Y3): now also G12.12 (A4)
- net at E5.5 (E1): now also E4.12 (Q2)
- net at G4.5 (A3): now also G3.8 (OUT)
- net at G4.6 (Y3): now also E4.2 (CP)
- net at D11.9 (A3): now also E10.3 (Y1)
- net at C7.5 (Q2): now also C6.10 (B3), C6.5 (B2)
- net ~{CPU-BRQ}: now reaches E4.1 (~{MR})
- net ~{CPU-BRQ}: now also U1.25 (~{BUSRQ})
- net CPU-CLK: now reaches U1.6 (~{CLK})
- net CPU-CLK: now also R41.1
- net at G11.13 (~{R2}): now also G12.11 (Y4)
- net at E10.1 (A1): now also E10.8 (Y3), R34.1
- net at E10.2 (B1): now also E10.6 (Y2)
- net at G12.13 (B4): now also G12.2 (B1), G12.8 (Y3)
- net at D9.3 (LPSTB): now also G10.9 (B1)
- net at C6.11 (Y4): now also C6.4 (A2)
- net at C6.3 (Y1): now also C6.9 (A3)
- net at G10.1 (B2): now also R37.1
- net at G10.10 (A0): now also R35.1, R36.2
- net at G10.3 (A=B): now also R33.1
- new net: J1.b6 (Pin_b6), JP1.1 (A)
- new net: JP1.2 (B), R35.2
- no-connect marks 0 -> 9
Other:
- moved on the sheet: C8

Commit message: Mainboard jumpers, keyboard IO, printer IO
Parts:
- added C1: C_Small, symbol Device:C_Small
- added C2, C3, C4, C5, C6, C7, C8, C9: 1nF, symbol Device:C_Small
- added J2: Conn_02x18_Counter_Clockwise, symbol Connector_Generic:Conn_02x18_Counter_Clockwise
- added J7: FG, symbol Connector:Conn_01x01_Pin
- added JP2: Jumper_2_Open, symbol Jumper:Jumper_2_Open
- added JP3: Jumper_2_Bridged, symbol Jumper:Jumper_2_Bridged
- added L1, L2, L3, L4, L5, L6, L7, L8: 100, symbol Device:L_Small
- added R1, R2: R_Network09, Resistor_THT:R_Array_SIP10, symbol Device:R_Network09
- added TP1: TestPoint, symbol Connector:TestPoint
- added uB2, uD1: 74LS74, symbol 74xx:74LS74
- added uD2, uF3: 74LS14, symbol 74xx:74LS04
- added uE1, uG1: 7407, symbol 74xx:74LS07
- added uF1: 10k, symbol Device:R_Pack08
- added uF2: 8255A, Package_DIP:DIP-40_W15.24mm, symbol Interface:8255A
- renumbered A1 to uA1, A2 to uA2, A3 to uA3, B1 to uB1, B3 to uB3, B4 to uB4, B5 to uB5, B6 to uB6, B7 to uB7, B8 to uB8, B9 to uB9, C10 to uC10, C11 to uC11, C12 to uC12, C13 to uC13, C3 to uC3, C4 to uC4, C5 to uC5, C6 to uC6, C7 to uC7, C8 to uC8, C9 to uC9, D10 to uD10, D11 to uD11, D12 to uD12, D13 to uD13, F4 to uD3, D4 to uD4, D5 to uD5, D6 to uD6, D7 to uD7, D8 to uD8, D9 to uD9, E10 to uE10, E11 to uE11, E12 to uE12, E13 to uE13, E4 to uE4, E5 to uE5, E6 to uE6, E7 to uE7, E8 to uE8, F10 to uF10, F11 to uF11, F12 to uF12, F13 to uF13, F6 to uF6, F7 to uF7, F8 to uF8, F9 to uF9, G10 to uG10, G11 to uG11, G12 to uG12, G3 to uG3, G4 to uG4, G9 to uG9, U1 to uU1
Connections:
- net BUS-A11: now also JP2.2 (B)
- net BUS-A15: now also uD11.10 (B3), uE10.10 (B3)
- net BUS-MREQ: now also uE10.12 (A4)
- net GND: now also J1.a5 (Pin_a5), J1.a6 (Pin_a6), J1.a8 (Pin_a8), uG3.7 (GND), uG4.7 (GND), J2.19 (Pin_19), J2.20 (Pin_20), J2.21 (Pin_21), J2.22 (Pin_22), J2.23 (Pin_23), J2.24 (Pin_24), J2.25 (Pin_25), J2.26 (Pin_26), J2.27 (Pin_27), J2.28 (Pin_28), J2.29 (Pin_29), TP1.1, uE1.7 (GND), uF3.7 (GND), uG1.7 (GND)
- net VCC: now also J1.b8 (Pin_b8), uE11.14 (VCC), uG3.14 (Vcc), uG4.14 (VCC), JP3.2 (B), R1.1 (common), R2.1 (common), uE1.14 (VCC), uF3.14 (VCC), uG1.14 (VCC); no longer uB9.21 (Vpp)
- net ~{BUS-IORD}: now also uC9.10 (B3), uF11.1 (A1)
- net ~{IO-Cycle}: now reaches uF11.11 (Y4)
- net ~{IO-Cycle}: now also uF11.4 (A2), uF11.5 (B2)
- net IO-Cycle: now reaches uF11.12 (A4)
- net IO-Cycle: now also uF11.13 (B4), uF11.3 (Y1)
- net CRTC-RS: now reaches uF11.6 (Y2)
- net CRTC-RS: now also uD9.24 (RS)
- net at uF11.8 (Y3): now also uF10.8 (A3), uF10.9 (B3)
- net at uF10.10 (Y3): now also uG11.10 (~{S2})
- net ~{IO-RST}: now reaches uF10.4 (Y2)
- net ~{IO-RST}: now also uD3.19 (~{MR}), uD9.2 (~{RESET})
- net at J1.a1 (Pin_a1): now also L1.1
- net at J1.a2 (Pin_a2): now also L3.1
- net at J1.a3 (Pin_a3): now also L5.1
- net at J1.a4 (Pin_a4): now also L7.1
- net at J1.a7 (Pin_a7): now also J7.1 (Pin_1)
- net at J1.b1 (Pin_b1): now also L2.1
- net at J1.b2 (Pin_b2): now also L4.1
- net at J1.b3 (Pin_b3): now also L6.1
- net at J1.b4 (Pin_b4): now also L8.1
- net ~{ROM-CE}: now reaches uD10.9 (3A), uD11.8 (Y3)
- net ~{ROM-CE}: now also uB9.18 (~{CE}/PGM)
- net at uD11.9 (A3), uE10.3 (Y1): now also uE10.4 (A2)
- net CPU-RFSH: now reaches uD10.12 (1Y)
- net CPU-RFSH: now also uE10.13 (B4)
- net at uG11.9 (Q2): now also uG1.1 (A1)
- new net: C2.1, L1.2
- new net: C2.2, R2.2 (R1), uF1.8 (R8.1)
- new net: C3.1, L2.2
- new net: C3.2, R2.3 (R2), uF1.7 (R7.1)
- new net: C5.1, L4.2
- new net: C5.2, R2.5 (R4), uF1.5 (R5.1)
- new net: C7.1, L6.2
- new net: C8.1, L7.2
- new net: C8.2, R2.8 (R7), uF1.2 (R2.1)
- new net: C4.1, L3.2
- new net: C6.1, L5.2
- new net: C4.2, R2.4 (R3), uF1.6 (R6.1)
- new net: C7.2, R2.7 (R6), uF1.3 (R3.1)
- new net: C6.2, R2.6 (R5), uF1.4 (R4.1)
- new net: C9.2, R2.9 (R8), uF1.1 (R1.1)
- new net: JP2.1 (A), JP3.1 (A), uB9.21 (Vpp)
- new net: C9.1, L8.2
- new net LPT-ACK: J2.10 (Pin_10)
- new net LPT-BUSY: J2.11 (Pin_11)
- new net LPT-DATA1: J2.2 (Pin_2), R1.2 (R1), uE1.10 (Y5)
- new net LPT-DATA2: J2.3 (Pin_3), R1.10 (R9), uE1.12 (Y6)
- new net LPT-DATA3: J2.4 (Pin_4), R1.3 (R2), uE1.8 (Y4)
- new net LPT-DATA4: J2.5 (Pin_5), R1.4 (R3), uG1.8 (Y4)
- new net LPT-DATA5: J2.6 (Pin_6), R1.5 (R4), uG1.6 (Y3)
- new net LPT-DATA6: J2.7 (Pin_7), R1.6 (R5), uG1.10 (Y5)
- new net LPT-DATA7: J2.8 (Pin_8), R1.7 (R6), uG1.4 (Y2)
- new net LPT-DATA8: J2.9 (Pin_9), R1.8 (R7), uG1.12 (Y6)
- new net LPT-LPSTB: J2.1 (Pin_1), uG1.2 (Y1)
- new net PPI-PA0: uF1.9 (R8.2), uF2.4 (PA0)
- new net PPI-PA1: uF1.10 (R7.2), uF2.3 (PA1)
- new net PPI-PA2: uF1.11 (R6.2), uF2.2 (PA2)
- new net PPI-PA3: uF1.12 (R5.2), uF2.1 (PA3)
- new net PPI-PA4: uF1.13 (R4.2), uF2.40 (PA4)
- new net PPI-PA5: uF1.14 (R3.2), uF2.39 (PA5)
- new net PPI-PA6: uF1.15 (R2.2), uF2.38 (PA6)
- new net PPI-PA7: uF1.16 (R1.2), uF2.37 (PA7)
- new net PPI-PB0: uE1.11 (A5), uF2.18 (PB0)
- new net PPI-PB1: uE1.13 (A6), uF2.19 (PB1)
- new net PPI-PB2: uE1.9 (A4), uF2.20 (PB2)
- new net PPI-PB3: uF2.21 (PB3), uG1.9 (A4)
- new net PPI-PB4: uF2.22 (PB4), uG1.5 (A3)
- new net PPI-PB5: uF2.23 (PB5), uG1.11 (A5)
- new net PPI-PB6: uF2.24 (PB6), uG1.3 (A2)
- new net PPI-PB7: uF2.25 (PB7), uG1.13 (A6)
- no-connect marks 9 -> 26
Other:
- moved on the sheet: J1

Commit message: Mainboard VRAM & CRAM addressing
Parts:
- added C10: 10nF, symbol Device:C_Small
- added C20: 10uF, symbol Device:C_Polarized_Small_US
- added C22: 10u, symbol Device:C_Polarized_Small
- added R27: 3R, symbol Device:R_Small_US
- added R28: 12k, symbol Device:R_Small_US
- added R32: 3k3, symbol Device:R_Small_US
- added R38, R39, R40: 1k, symbol Device:R_Small_US
- added uF4: 74LS166, symbol 74xx:74LS166
- uG10: value MC14585 -> MC14584
Connections:
- net GND: now also uD4.10 (GND), uD5.10 (GND), uD6.8 (GND), uD7.10 (GND), uD8.8 (GND), uD9.1 (GND), uE4.8 (GND), uE5.7 (GND), uE6.8 (GND), uE7.10 (GND), uE8.8 (GND), uF6.12 (GND), uF7.8 (GND), uF8.12 (GND), uF8.18 (~{CE}), uG10.7 (Vss), C20.2, uF4.8 (GND); no longer uG10.8 (Vss)
- net VCC: now also uC5.14 (VCC), uD4.20 (VCC), uD5.20 (VCC), uD6.16 (VCC), uD7.20 (VCC), uD8.16 (VCC), uD9.20 (VCC), uE4.16 (VCC), uE5.14 (VCC), uE6.16 (VCC), uE7.20 (VCC), uE8.16 (VCC), uF6.24 (Vcc), uF7.16 (VCC), uF8.24 (Vcc), uF9.16 (VCC), uG10.14 (Vdd), R28.2, R32.2, R38.2, R39.2, R40.2, uF4.16 (VCC); no longer uG10.16 (Vdd)
- net ~{BUS-WR}: now also R40.1
- net ~{CPU-RST}: now also uG10.13 (A6); no longer uG10.15 (A3)
- net ~{MEM-CAS}: now also R38.1
- net ~{MEM-RAS}: now also R39.1
- net LPT-STROBE: now reaches uG1.1 (A1), uG11.9 (Q2)
- net ~{LPT-CE}: now reaches uB6.15 (O0), uG12.9 (A3)
- net VRAM-AMUX: now reaches uC6.8 (Y3), uD8.1 (S), uE8.1 (S), uF9.1 (S)
- net CRTC-MA6: now reaches uE8.10 (I1c)
- net CRTC-MA6: now also uD9.10 (MA6)
- net VRAM-A4: now reaches uE8.12 (Zd)
- net VRAM-A4: now also uF8.4 (A4)
- net CRTC-MA4: now reaches uE8.14 (I0d)
- net CRTC-MA4: now also uD9.8 (MA4)
- net CRTC-MA5: now reaches uE8.3 (I1a)
- net CRTC-MA5: now also uD9.9 (MA5)
- net VRAM-A5: now reaches uE8.4 (Za)
- net VRAM-A5: now also uF8.3 (A5)
- net CRTC-MA7: now reaches uE8.6 (I1b)
- net CRTC-MA7: now also uD9.11 (MA7)
- net VRAM-A7: now reaches uE8.7 (Zb)
- net VRAM-A7: now also uF8.1 (A7)
- net VRAM-A6: now reaches uE8.9 (Zc)
- net VRAM-A6: now also uF8.2 (A6)
- net CRTC-RA3: now reaches uC5.11 (A5)
- net CRTC-RA3: now also uD9.35 (RA3)
- net VRAM-D1: now reaches uF8.10 (Q1)
- net VRAM-D1: now also uD7.3 (O3b), uE7.4 (D1)
- net VRAM-D2: now reaches uF8.11 (Q2)
- net VRAM-D2: now also uD7.16 (O1a), uE7.17 (D6)
- net VRAM-D3: now reaches uF8.13 (Q3)
- net VRAM-D3: now also uD7.5 (O2b), uE7.14 (D5)
- net VRAM-D4: now reaches uF8.14 (Q4)
- net VRAM-D4: now also uD7.14 (O2a), uE7.7 (D2)
- net VRAM-D5: now reaches uF8.15 (Q5)
- net VRAM-D5: now also uD7.7 (O1b), uE7.8 (D3)
- net VRAM-D6: now reaches uF8.16 (Q6)
- net VRAM-D6: now also uD7.12 (O3a), uE7.13 (D4)
- net VRAM-D7: now reaches uF8.17 (Q7)
- net VRAM-D7: now also uD7.9 (O0b), uE7.18 (D7)
- net VRAM-A10: now reaches uF8.19 (A10)
- net VRAM-A10: now also uF9.9 (Zc)
- net VRAM-A9: now reaches uF8.22 (A9)
- net VRAM-A9: now also uF9.12 (Zd)
- net VRAM-A8: now reaches uF8.23 (A8)
- net VRAM-A8: now also uF9.4 (Za)
- net VRAM-A3: now reaches uF8.5 (A3)
- net VRAM-A3: now also uD8.12 (Zd)
- net VRAM-A2: now reaches uF8.6 (A2)
- net VRAM-A2: now also uD8.4 (Za)
- net VRAM-A1: now reaches uF8.7 (A1)
- net VRAM-A1: now also uD8.7 (Zb)
- net VRAM-A0: now reaches uF8.8 (A0)
- net VRAM-A0: now also uD8.9 (Zc)
- net VRAM-D0: now reaches uF8.9 (Q0)
- net VRAM-D0: now also uD7.18 (O0a), uE7.3 (D0)
- net at uF10.8 (A3), uF10.9 (B3), uF11.8 (Y3): now also C22.1
- net CRAM-A7: now reaches uF6.1 (A7)
- net CRAM-A7: now also uE6.7 (Zb)
- net CRAM-D1: now reaches uF6.10 (Q1)
- net CRAM-D1: now also uF4.3 (B)
- net CRAM-D2: now reaches uF6.11 (Q2)
- net CRAM-D2: now also uF4.4 (C)
- net CRAM-D3: now reaches uF6.13 (Q3)
- net CRAM-D3: now also uF4.5 (D)
- net CRAM-D4: now reaches uF6.14 (Q4)
- net CRAM-D4: now also uF4.10 (E)
- net CRAM-D5: now reaches uF6.15 (Q5)
- net CRAM-D5: now also uF4.11 (F)
- net CRAM-D6: now reaches uF6.16 (Q6)
- net CRAM-D6: now also uF4.12 (G)
- net CRAM-D7: now reaches uF6.17 (Q7)
- net CRAM-D7: now also uF4.14 (H)
- net CRAM-A10: now reaches uF6.19 (A10)
- net CRAM-A10: now also uF7.9 (Zc)
- net CRAM-A6: now reaches uF6.2 (A6)
- net CRAM-A6: now also uE6.9 (Zc)
- net CRAM-A9: now reaches uF6.22 (A9)
- net CRAM-A9: now also uF7.12 (Zd)
- net CRAM-A8: now reaches uF6.23 (A8)
- net CRAM-A8: now also uF7.4 (Za)
- net CRAM-A5: now reaches uF6.3 (A5)
- net CRAM-A5: now also uE6.4 (Za)
- net CRAM-A4: now reaches uF6.4 (A4)
- net CRAM-A4: now also uE6.12 (Zd)
- net CRAM-A3: now reaches uF6.5 (A3)
- net CRAM-A3: now also uD6.12 (Zd)
- net CRAM-A2: now reaches uF6.6 (A2)
- net CRAM-A2: now also uD6.4 (Za)
- net CRAM-A1: now reaches uF6.7 (A1)
- net CRAM-A1: now also uD6.7 (Zb)
- net CRAM-A0: now reaches uF6.8 (A0)
- net CRAM-A0: now also uD6.9 (Zc)
- net CRAM-D0: now reaches uF6.9 (Q0)
- net CRAM-D0: now also uF4.2 (A)
- net MEM-AMUX: now reaches uC10.1 (S)
- net MEM-AMUX: now also uC11.1 (S), uD10.8 (3Y), uE11.13 (A6)
- net at R35.1, R36.2: now also uG10.9 (A4); no longer uG10.10 (A0)
- net at uA2.10 (I4), uB8.17 (I3b), uE4.13 (Q1)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: now also uC7.9 (C2)
- net CRAM-AMUX: now reaches uC6.6 (Y2), uD6.1 (S), uE6.1 (S), uF7.1 (S)
- net VRAM-D7R: now reaches uF7.10 (I1c)
- net VRAM-D7R: now also uE7.19 (O7)
- net VRAM-D6R: now reaches uF7.14 (I0d)
- net VRAM-D6R: now also uE7.12 (O4)
- net VRAM-D5R: now reaches uF7.3 (I1a)
- net VRAM-D5R: now also uE7.9 (O3)
- net at R37.1, uG10.1 (A1): now also C22.2
- net at J1.b7 (Pin_b7): now also R27.1
- net at uG9.13 (~{R2}): now also uF3.8 (Y4)
- net at uG9.8 (~{Q2}): now also C10.1, R32.1
- net IO-D7: now reaches uD7.11 (I0b)
- net IO-D7: now also uD5.11 (B7), uD9.26 (D7)
- net IO-D5: now reaches uD7.13 (I1b)
- net IO-D5: now also uD5.13 (B5), uD9.28 (D5)
- net IO-D3: now reaches uD7.15 (I2b)
- net IO-D3: now also uD5.15 (B3), uD9.30 (D3)
- net IO-D1: now reaches uD7.17 (I3b)
- net IO-D1: now also uD5.17 (B1), uD9.32 (D1)
- net IO-D0: now reaches uD7.2 (I0a)
- net IO-D0: now also uD5.18 (B0), uD9.33 (D0)
- net IO-D2: now reaches uD7.4 (I1a)
- net IO-D2: now also uD5.16 (B2), uD9.31 (D2)
- net IO-D4: now reaches uD7.6 (I2a)
- net IO-D4: now also uD5.14 (B4), uD9.29 (D4)
- net IO-D6: now reaches uD7.8 (I3a)
- net IO-D6: now also uD5.12 (B6), uD9.27 (D6)
- net at uF3.9 (A4): now also C20.1, R27.2, R28.1
- net CRTC-MA10: now reaches uF9.10 (I1c)
- net CRTC-MA10: now also uD9.14 (MA10)
- net CRTC-MA9: now reaches uF9.14 (I0d)
- net CRTC-MA9: now also uD9.13 (MA9)
- net CRTC-MA8: now reaches uF9.3 (I1a)
- net CRTC-MA8: now also uD9.12 (MA8)
- net ~{LPT-WR}: now reaches uG12.13 (B4), uG12.2 (B1), uG12.8 (Y3)
- net VRAM-D3R: now reaches uE7.15 (O5)
- net VRAM-D3R: now also uE6.10 (I1c)
- net VRAM-D2R: now reaches uE7.16 (O6)
- net VRAM-D2R: now also uE6.3 (I1a)
- net VRAM-D0R: now reaches uE7.2 (O0)
- net VRAM-D1R: now reaches uE7.5 (O1)
- net VRAM-D1R: now also uE6.14 (I0d)
- net VRAM-D4R: now reaches uE7.6 (O2)
- net VRAM-D4R: now also uE6.6 (I1b)
- net at uD9.3 (LPSTB): now also uG10.8 (Y4); no longer uG10.9 (B1)
- net CRTC-RA2: now reaches uD9.36 (RA2)
- net CRTC-RA2: now also uD6.3 (I1a)
- net CRTC-RA1: now reaches uD9.37 (RA1)
- net CRTC-RA1: now also uD6.6 (I1b)
- net CRTC-RA0: now reaches uD9.38 (RA0)
- net CRTC-RA0: now also uD6.10 (I1c)
- net CRTC-MA0: now reaches uD9.4 (MA0)
- net CRTC-MA0: now also uD8.10 (I1c)
- net CRTC-MA1: now reaches uD9.5 (MA1)
- net CRTC-MA1: now also uD8.6 (I1b)
- net CRTC-MA2: now reaches uD9.6 (MA2)
- net CRTC-MA2: now also uD8.3 (I1a)
- net CRTC-MA3: now reaches uD9.7 (MA3)
- net CRTC-MA3: now also uD8.14 (I0d)
- net at R33.1, uG10.3 (A2): now also C10.2
- no-connect marks 26 -> 50
Other:
- note added: "CHAR RAM"
- note added: "Video RAM"
- moved on the sheet: R33, R34, R36, R37, uE6
