File: Mainboard/MBC-1000_Mainboard/MBC-1000_Mainboard.kicad_sch (KiCad schematic)
At the start: 108 parts, among them J1 Keyboard, J2 Conn_02x18_Counter_Clockwise, J7 FG, U2 74LS32

Commit message: add info on disks, monitor, serial, keyboard pinout
Connections:
- net GND: now also J1.b5 (Pin_b5), J1.b6 (Pin_b6), J1.b8 (Pin_b8); no longer J1.a5 (Pin_a5), J1.a6 (Pin_a6), J1.a8 (Pin_a8)
- net VCC: now also J1.a8 (Pin_a8); no longer J1.b8 (Pin_b8)
- net at J1.b7 (Pin_b7): now also J7.1 (Pin_1); no longer R27.1
- net KEY-D2: now reaches J1.b2 (Pin_b2)
- net KEY-D2: now also L3.1; no longer L4.1
- net KEY-D4: now reaches J1.b3 (Pin_b3)
- net KEY-D4: now also L5.1; no longer L6.1
- net KEY-D0: now reaches L1.1
- net KEY-D0: now also J1.b1 (Pin_b1); no longer J1.a1 (Pin_a1)
- net KEY-D3: now reaches J1.a2 (Pin_a2)
- net KEY-D3: now also L4.1; no longer L3.1
- net KEY-D5: now reaches J1.a3 (Pin_a3)
- net KEY-D5: now also L6.1; no longer L5.1
- net KEY-D6: now reaches L7.1
- net KEY-D6: now also J1.b4 (Pin_b4); no longer J1.a4 (Pin_a4)
- net KEY-REST: now reaches J1.a7 (Pin_a7)
- net KEY-REST: now also R27.1; no longer J7.1 (Pin_1)
- net KEY-D1: now reaches L2.1
- net KEY-D1: now also J1.a1 (Pin_a1); no longer J1.b1 (Pin_b1)
- net KEY-D7: now reaches L8.1
- net KEY-D7: now also J1.a4 (Pin_a4); no longer J1.b4 (Pin_b4)
- net ~{KEY-LPSB}: now reaches JP1.1 (A)
- net ~{KEY-LPSB}: now also J1.a6 (Pin_a6); no longer J1.b6 (Pin_b6)
Other:
- note added: "Character RAM"
- note removed: "CHAR RAM"
- moved on the sheet: J1
Changed lines of the file:
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@@
 	(wire
 		(pts
-			(xy 302.26 264.16) (xy 302.26 299.72)
+			(xy 294.64 264.16) (xy 294.64 299.72)
 		)
 		(stroke
@@
 	(wire
 		(pts
+			(xy 330.2 271.78) (xy 365.76 271.78)
+		)
+		(stroke
+			(width 0)
+			(type default)
+		)
+	)
+	(wire
+		(pts
 			(xy 942.34 71.12) (xy 952.5 71.12)
 		)
@@
 	(wire
 		(pts
-			(xy 363.22 292.1) (xy 307.34 292.1)
+			(xy 363.22 292.1) (xy 299.72 292.1)
 		)
 		(stroke
@@
 	(wire
 		(pts
-			(xy 312.42 276.86) (xy 312.42 287.02)
+			(xy 304.8 276.86) (xy 304.8 287.02)
 		)
 		(stroke
@@
 	(wire
 		(pts
-			(xy 309.88 289.56) (xy 309.88 274.32)
+			(xy 302.26 289.56) (xy 302.26 274.32)
 		)
 		(stroke
@@
 	(wire
 		(pts
-			(xy 309.88 274.32) (xy 317.5 274.32)
+			(xy 302.26 274.32) (xy 317.5 274.32)
 		)
 		(stroke
@@
 	(wire
 		(pts
-			(xy 304.8 266.7) (xy 304.8 304.8)
+			(xy 297.18 266.7) (xy 297.18 304.8)
 		)
 		(stroke
@@
 	(wire
 		(pts
-			(xy 307.34 292.1) (xy 307.34 271.78)
+			(xy 299.72 292.1) (xy 299.72 271.78)
 		)
 		(stroke
@@
 	(wire
 		(pts
-			(xy 312.42 287.02) (xy 373.38 287.02)
+			(xy 304.8 287.02) (xy 373.38 287.02)
 		)
 		(stroke
@@
 	(wire
 		(pts
-			(xy 302.26 299.72) (xy 635 299.72)
+			(xy 294.64 299.72) (xy 635 299.72)
 		)
 		(stroke
@@
 	(wire
 		(pts
-			(xy 375.92 276.86) (xy 330.2 276.86)
+			(xy 840.74 93.98) (xy 850.9 93.98)
 		)
 		(stroke
@@
 	(wire
 		(pts
-			(xy 840.74 93.98) (xy 850.9 93.98)
+			(xy 825.5 210.82) (xy 835.66 210.82)
 		)
 		(stroke
@@
 	(wire
 		(pts
-			(xy 825.5 210.82) (xy 835.66 210.82)
+			(xy 723.9 137.16) (xy 736.6 137.16)
 		)
 		(stroke
@@
 	(wire
 		(pts
-			(xy 723.9 137.16) (xy 736.6 137.16)
+			(xy 431.8 248.92) (xy 444.5 248.92)
 		)
 		(stroke
@@
 	(wire
 		(pts
-			(xy 431.8 248.92) (xy 444.5 248.92)
+			(xy 622.3 241.3) (xy 632.46 241.3)
 		)
 		(stroke
@@
 	(wire
 		(pts
-			(xy 622.3 241.3) (xy 632.46 241.3)
+			(xy 330.2 274.32) (xy 370.84 274.32)
 		)
 		(stroke
@@
 	(wire
 		(pts
-			(xy 304.8 304.8) (xy 520.7 304.8)
+			(xy 297.18 304.8) (xy 520.7 304.8)
 		)
 		(stroke
@@
 	(wire
 		(pts
-			(xy 317.5 276.86) (xy 312.42 276.86)
+			(xy 317.5 276.86) (xy 304.8 276.86)
 		)
 		(stroke
@@
 	(wire
 		(pts
-			(xy 314.96 284.48) (xy 378.46 284.48)
+			(xy 307.34 284.48) (xy 378.46 284.48)
 		)
 		(stroke
@@
 	(wire
 		(pts
+			(xy 330.2 276.86) (xy 375.92 276.86)
+		)
+		(stroke
+			(width 0)
+			(type default)
+		)
+	)
+	(wire
+		(pts
 			(xy 876.3 187.96) (xy 886.46 187.96)
 		)
@@
 	(wire
 		(pts
-			(xy 317.5 266.7) (xy 304.8 266.7)
+			(xy 317.5 266.7) (xy 297.18 266.7)
 		)
 		(stroke
@@
 	(wire
 		(pts
-			(xy 365.76 271.78) (xy 330.2 271.78)
-		)
-		(stroke
-			(width 0)
-			(type default)
-		)
-	)
-	(wire
-		(pts
 			(xy 840.74 193.04) (xy 850.9 193.04)
 		)
@@
 	(wire
 		(pts
-			(xy 314.96 279.4) (xy 314.96 284.48)
+			(xy 307.34 279.4) (xy 307.34 284.48)
 		)
 		(stroke
@@
 	(wire
 		(pts
-			(xy 307.34 271.78) (xy 317.5 271.78)
+			(xy 299.72 271.78) (xy 317.5 271.78)
 		)
 		(stroke
@@
 	(wire
 		(pts
-			(xy 317.5 264.16) (xy 302.26 264.16)
+			(xy 317.5 264.16) (xy 294.64 264.16)
 		)
 		(stroke
@@
 	(wire
 		(pts
-			(xy 370.84 274.32) (xy 330.2 274.32)
-		)
-		(stroke
-			(width 0)
-			(type default)
-		)
-	)
-	(wire
-		(pts
 			(xy 1028.7 208.28) (xy 1038.86 208.28)
 		)
@@
 	(wire
 		(pts
-			(xy 317.5 279.4) (xy 314.96 279.4)
+			(xy 317.5 279.4) (xy 307.34 279.4)
 		)
 		(stroke
@@
 	(wire
 		(pts
-			(xy 368.3 289.56) (xy 309.88 289.56)
+			(xy 368.3 289.56) (xy 302.26 289.56)
 		)
 		(stroke
@@
 		)
 	)
-	(text "CHAR RAM"
+	(text "Character RAM"
 		(exclude_from_sim no)
 		(at 711.2 264.16 0)
@@
 		)
 	)
+	(label "~{KEY-STB}"
+		(at 307.34 269.24 0)
+		(fields_autoplaced yes)
+		(effects
+			(font
+				(size 1.27 1.27)
+			)
+			(justify left bottom)
+		)
+	)
 	(label "CPU-A9"
 		(at 1038.86 63.5 180)
@@
 		)
 	)
+	(label "KEY-D1"
+		(at 307.34 279.4 0)
+		(fields_autoplaced yes)
+		(effects
+			(font
+				(size 1.27 1.27)
+			)
+			(justify left bottom)
+		)
+	)
 	(label "CPU-D3"
 		(at 1043.94 162.56 0)
@@
 		)
 	)
+	(label "KEY-D4"
+		(at 337.82 274.32 180)
+		(fields_autoplaced yes)
+		(effects
+			(font
+				(size 1.27 1.27)
+			)
+			(justify right bottom)
+		)
+	)
 	(label "~{CPU-MREQ}"
 		(at 891.54 236.22 0)
@@
 		)
 	)
+	(label "KEY-D0"
+		(at 337.82 279.4 180)
+		(fields_autoplaced yes)
+		(effects
+			(font
+				(size 1.27 1.27)
+			)
+			(justify right bottom)
+		)
+	)
 	(label "CRTC-MA8"
 		(at 840.74 236.22 0)
@@
 		)
 	)
+	(label "KEY-D5"
+		(at 307.34 274.32 0)
+		(fields_autoplaced yes)
+		(effects
+			(font
+				(size 1.27 1.27)
+			)
+			(justify left bottom)
+		)
+	)
 	(label "~{CPU-BRQ}"
 		(at 586.74 195.58 0)
@@
 		)
 	)
+	(label "KEY-D6"
+		(at 337.82 271.78 180)
+		(fields_autoplaced yes)
+		(effects
+			(font
+				(size 1.27 1.27)
+			)
+			(justify right bottom)
+		)
+	)
 	(label "~{MEM-RAS}"
 		(at 993.14 203.2 0)
@@
 		)
 	)
+	(label "KEY-D3"
+		(at 307.34 276.86 0)
+		(fields_autoplaced yes)
+		(effects
+			(font
+				(size 1.27 1.27)
+			)
+			(justify left bottom)
+		)
+	)
 	(label "MEM-A2"
 		(at 891.54 142.24 0)
@@
 		)
 	)
+	(label "KEY-D7"
+		(at 307.34 271.78 0)
+		(fields_autoplaced yes)
+		(effects
+			(font
+				(size 1.27 1.27)
+			)
+			(justify left bottom)
+		)
+	)
 	(label "BUS-A7"
 		(at 937.26 73.66 180)
@@
 		)
 	)
+	(label "KEY-REST"
+		(at 307.34 264.16 0)
+		(fields_autoplaced yes)
+		(effects
+			(font
+				(size 1.27 1.27)
+			)
+			(justify left bottom)
+		)
+	)
 	(label "MEM-A4"
 		(at 1038.86 243.84 180)
@@
 		)
 	)
+	(label "~{KEY-LPSB}"
+		(at 307.34 266.7 0)
+		(fields_autoplaced yes)
+		(effects
+			(font
+				(size 1.27 1.27)
+			)
+			(justify left bottom)
+		)
+	)
 	(label "CPU-D0"
 		(at 993.14 93.98 0)
@@
 		)
 	)
+	(label "KEY-D2"
+		(at 337.82 276.86 180)
+		(fields_autoplaced yes)
+		(effects
+			(font
+				(size 1.27 1.27)
+			)
+			(justify right bottom)
+		)
+	)
 	(label "CRTC-MA2"
 		(at 840.74 172.72 0)
@@
 	(symbol
 		(lib_id "Connector_Generic:Conn_02x08_Row_Letter_First")
-		(at 325.12 271.78 180)
+		(at 322.58 271.78 0)
+		(mirror x)
 		(unit 1)
 		(exclude_from_sim no)
@@
 		(on_board yes)
 		(dnp no)
-		(fields_autoplaced yes)
 		(property "Reference" "J1"
 			(at 323.85 256.2055 0)
@@
 		)
 		(property "Footprint" ""
-			(at 325.12 271.78 0)
+			(at 322.58 271.78 0)
 			(effects
 				(font
@@
 		)
 		(property "Datasheet" "~"
-			(at 325.12 271.78 0)
+			(at 322.58 271.78 0)
 			(effects
 				(font
@@
 		)
 		(property "Description" "Generic connector, double row, 02x08, row letter first pin numbering scheme (pin number consists of a letter for the row and a number for the pin index in this row. a1, ..., aN; b1, ..., bN), script generated (kicad-library-utils/schlib/autogen/connector/)"
-			(at 325.12 271.78 0)
+			(at 322.58 271.78 0)
 			(effects
 				(font

Commit message: Add remaining IC & connector footprints to mainboard schematic
Parts:
- added BZ1: Buzzer, symbol Device:Buzzer
- added J3: Conn_01x08, symbol Connector_Generic:Conn_01x08
- added J4: Conn_02x17_Odd_Even, symbol Connector_Generic:Conn_02x17_Odd_Even
- added J6: Conn_02x25_Odd_Even, symbol Connector_Generic:Conn_02x25_Odd_Even
- added uA1: RC4558, symbol Amplifier_Operational:RC4558
- added uA2, uC2: 74LS221, symbol 74xx:74LS221
- added uB1: 74166, symbol 74xx:74LS166
- added uC0: SN75452B, symbol MBC-1000_Mainboard:SN75452B
- added uC1: 74145, symbol 74xx:74LS145
- added uE2: 74LS123, symbol 74xx:74LS123
Connections:
- net GND: now also J3.5 (Pin_5), J3.6 (Pin_6)
- net VCC: now also J3.1 (Pin_1), J3.3 (Pin_3), J3.4 (Pin_4)
- new net +12V: J3.7 (Pin_7), uC0.8 (Vcc)
- no-connect marks 50 -> 51

Commit message: Mainboard clock & expansion bus
Parts:
- added R3, R4, R44, R45: 3k3, symbol Device:R_Small_US
Connections:
- net CPU-CLK: now also uA2.9 (O4a), uF10.11 (A4)
- net GND: now also J6.10 (Pin_10), J6.12 (Pin_12), J6.14 (Pin_14), J6.16 (Pin_16), J6.18 (Pin_18), J6.2 (Pin_2), J6.20 (Pin_20), J6.22 (Pin_22), J6.24 (Pin_24), J6.26 (Pin_26), J6.28 (Pin_28), J6.30 (Pin_30), J6.32 (Pin_32), J6.34 (Pin_34), J6.36 (Pin_36), J6.38 (Pin_38), J6.4 (Pin_4), J6.40 (Pin_40), J6.42 (Pin_42), J6.44 (Pin_44), J6.6 (Pin_6), J6.8 (Pin_8)
- net VCC: now also J6.46 (Pin_46), J6.48 (Pin_48), J6.50 (Pin_50), uE4.10 (CET), uE4.7 (CEP), uE4.9 (~{PE}), R44.1, R45.1
- net ~{CPU-RFSH}: no longer uB8.15 (I2b)
- net ~{CPU-RST}: now also uB8.15 (I2b)
- net ~{CLK-16M}: now reaches uG3.8 (OUT), uG4.5 (A3)
- net EXP-D7: now reaches uB5.2 (A0)
- net EXP-D7: now also J6.15 (Pin_15)
- net EXP-D6: now reaches uB5.3 (A1)
- net EXP-D6: now also J6.13 (Pin_13)
- net EXP-D5: now reaches uB5.4 (A2)
- net EXP-D5: now also J6.11 (Pin_11)
- net EXP-D4: now reaches uB5.5 (A3)
- net EXP-D4: now also J6.9 (Pin_9)
- net EXP-D3: now reaches uB5.6 (A4)
- net EXP-D3: now also J6.7 (Pin_7)
- net EXP-D2: now reaches uB5.7 (A5)
- net EXP-D2: now also J6.5 (Pin_5)
- net EXP-D1: now reaches uB5.8 (A6)
- net EXP-D1: now also J6.3 (Pin_3)
- net EXP-D0: now reaches uB5.9 (A7)
- net EXP-D0: now also J6.1 (Pin_1)
- net ~{EXT-M1}: now reaches uB8.12 (O3a)
- net ~{EXT-M1}: now also J6.47 (Pin_47)
- net ~{EXP-IORQ}: now reaches uB8.14 (O2a)
- net ~{EXP-IORQ}: now also J6.45 (Pin_45)
- net CLK-4M: now reaches uA2.10 (I4), uB8.17 (I3b), uC7.9 (C2), uE4.13 (Q1), uE5.4 (D1)
- net EXT-CLK: now reaches uB8.3 (O3b)
- net EXT-CLK: now also J6.39 (Pin_39)
- net ~{EXT-RST}: now reaches uB8.5 (O2b)
- net ~{EXT-RST}: now also J6.37 (Pin_37)
- net EXP-A7: now reaches uB8.7 (O1b)
- net EXP-A7: now also J6.35 (Pin_35)
- net EXP-A6: now reaches uB8.9 (O0b)
- net EXP-A6: now also J6.33 (Pin_33)
- net CLK-8M: now reaches uE5.2 (B1)
- net CLK-8M: now also uE4.14 (Q0)
- net CLK-2M: now reaches uE4.12 (Q2), uE5.5 (E1)
- net CLK-16M: now reaches uE4.2 (CP), uG4.6 (Y3)
- net ~{CPU-INT}: now reaches uU1.16 (~{INT})
- net ~{CPU-INT}: now also R3.2
- net ~{CPU-NMI}: now reaches uU1.17 (~{NMI})
- net ~{CPU-NMI}: now also R4.2
- net ~{EXP-WR}: now reaches J6.17 (Pin_17)
- net ~{EXP-WR}: now also uB7.9 (O0b)
- net ~{EXP-RD}: now reaches J6.19 (Pin_19)
- net ~{EXP-RD}: now also uB7.7 (O1b)
- net EXP-A0: now reaches J6.21 (Pin_21)
- net EXP-A0: now also uB7.5 (O2b)
- net EXP-A1: now reaches J6.23 (Pin_23)
- net EXP-A1: now also uB7.3 (O3b)
- net EXP-A2: now reaches J6.25 (Pin_25)
- net EXP-A2: now also uB7.18 (O0a)
- net EXP-A3: now reaches J6.27 (Pin_27)
- net EXP-A3: now also uB7.16 (O1a)
- net EXP-A4: now reaches J6.29 (Pin_29)
- net EXP-A4: now also uB7.14 (O2a)
- net EXP-A5: now reaches J6.31 (Pin_31)
- net EXP-A5: now also uB7.12 (O3a)
- net ~{EXT-INT}: now reaches J6.41 (Pin_41)
- net ~{EXT-INT}: now also R3.1, R45.2
- net ~{EXT-NMI}: now reaches J6.43 (Pin_43)
- net ~{EXT-NMI}: now also R4.1, R44.2
- no-connect marks 51 -> 58

Commit message: Mainboard floppy interface, Video memory addressing
Parts:
- removed uB1: 74166, symbol 74xx:74LS166
- added C28: 1nF, symbol Device:C_Small
- added D1: D, symbol Device:D
- added Q1: D1111, symbol Device:Q_NPN_Darlington_ECB
- added R7, R8: 10k, symbol Device:R_Small_US
- added uB1: 7416, symbol 74xx_IEEE:7416
Connections:
- net BUS-A0: now also uD3.5 (A0), uF2.9 (A0), uF7.2 (I0a), uF9.2 (I0a)
- net BUS-A1: now also uD3.6 (A1), uF2.8 (A1), uF7.13 (I1d), uF9.13 (I1d)
- net BUS-A10: now also uD6.2 (I0a), uD8.2 (I0a)
- net BUS-A11: now also uD6.13 (I1d), uD8.13 (I1d)
- net BUS-A12: now also uE6.13 (I1d), uE8.13 (I1d)
- net BUS-A13: now also uE6.2 (I0a), uE8.2 (I0a)
- net BUS-A14: now also uE6.11 (I0c), uE8.11 (I0c)
- net BUS-A15: now also uE6.5 (I0b), uE8.5 (I0b)
- net BUS-A2: now also uF7.11 (I0c), uF9.11 (I0c)
- net BUS-A8: now also uD6.11 (I0c), uD8.11 (I0c)
- net BUS-A9: now also uD6.5 (I0b), uD8.5 (I0b)
- net CLK-2M: now also uC4.9 (A3), uC5.9 (A4), uE5.11 (G1)
- net CLK-4M: now also uE5.3 (C1), uG4.13 (A6)
- net CLK-8M: now also uE5.1 (A1)
- net CPU-D0: now also uB5.11 (B7), uD5.2 (A0)
- net CPU-D1: now also uB5.12 (B6), uD5.3 (A1)
- net CPU-D2: now also uB5.13 (B5), uD5.4 (A2)
- net CPU-D3: now also uB5.14 (B4), uD5.5 (A3)
- net CPU-D4: now also uB5.15 (B3), uD5.6 (A4)
- net CPU-D5: now also uB5.16 (B2), uD5.7 (A5)
- net CPU-D6: now also uB5.17 (B1), uD5.8 (A6)
- net CPU-D7: now also uB5.18 (B0), uD5.9 (A7)
- net CRAM-D0: now also uD4.18 (O0a)
- net CRAM-D1: now also uD4.3 (O3b)
- net CRAM-D2: now also uD4.16 (O1a)
- net CRAM-D3: now also uD4.5 (O2b)
- net CRAM-D4: now also uD4.14 (O2a)
- net CRAM-D5: now also uD4.7 (O1b)
- net CRAM-D6: now also uD4.12 (O3a)
- net CRAM-D7: now also uD4.9 (O0b)
- net GND: now also J4.1 (Pin_1), J4.11 (Pin_11), J4.13 (Pin_13), J4.15 (Pin_15), J4.17 (Pin_17), J4.19 (Pin_19), J4.2 (Pin_2), J4.21 (Pin_21), J4.23 (Pin_23), J4.25 (Pin_25), J4.27 (Pin_27), J4.29 (Pin_29), J4.3 (Pin_3), J4.31 (Pin_31), J4.33 (Pin_33), J4.4 (Pin_4), J4.5 (Pin_5), J4.7 (Pin_7), J4.9 (Pin_9), uA3.7 (GND), uB2.7 (GND), uB3.7 (GND), uB4.7 (GND), uB5.10 (GND), uB5.19 (CE), uC0.4 (GND), uC1.12 (P3), uC1.13 (P2), uC1.8 (GND), uC4.7 (GND), uC5.7 (GND), uC7.4 (K1), uD1.7 (GND), uD2.7 (GND), uD3.20 (GND), uD3.37 (~{DDEN}), uD5.19 (CE), uD6.15 (E), uD8.15 (E), uE6.15 (E), uE8.15 (E), uF2.7 (GND), uF6.18 (~{CE}), uF7.15 (E), uF9.15 (E), Q1.1 (E), uB1.7 (GND)
- net IO-D0: now also uD3.7 (DAL0), uD4.2 (I0a), uF2.34 (D0)
- net IO-D1: now also uD3.8 (DAL1), uD4.17 (I3b), uF2.33 (D1)
- net IO-D2: now also uD3.9 (DAL2), uD4.4 (I1a), uF2.32 (D2)
- net IO-D3: now also uD3.10 (DAL3), uD4.15 (I2b), uF2.31 (D3)
- net IO-D4: now also uD3.11 (DAL4), uD4.6 (I2a), uF2.30 (D4)
- net IO-D5: now also uD3.12 (DAL5), uD4.13 (I1b), uF2.29 (D5)
- net IO-D6: now also uD3.13 (DAL6), uD4.8 (I3a), uF2.28 (D6)
- net IO-D7: now also uD3.14 (DAL7), uD4.11 (I0b), uF2.27 (D7)
- net VCC: now also BZ1.1 (+), uA3.14 (VCC), uB2.14 (VCC), uB3.14 (VCC), uB4.14 (VCC), uB5.20 (VCC), uC1.16 (VCC), uC4.14 (VCC), uC7.1 (J1), uC7.10 (~{R2}), uD1.14 (VCC), uD2.14 (VCC), uD3.21 (Vcc), uD3.22 (~{TEST}), uF2.26 (VCC), uF4.9 (Clr), uF7.6 (I1b), uF9.6 (I1b), uU1.24 (~{WAIT}), uB1.14 (VCC)
- net ~{BUS-IORD}: now also uD3.4 (~{RE}), uF2.5 (~{RD})
- net ~{BUS-IOWR}: now also uD3.2 (~{WE}), uF2.36 (~{WR})
- net ~{CPU-IORQ}: now also uC8.3 (B1)
- net ~{CPU-M1}: now also uC8.2 (A1)
- net ~{CPU-RST}: now also uF3.1 (A1)
- net ~{PPI-CE}: now also uF2.6 (~{CS})
- net CPU-INTAK: now reaches uC9.4 (A2)
- net CPU-INTAK: now also uC8.1 (Y1)
- net EXP-DIR: now reaches uC9.6 (Y2)
- net EXP-DIR: now also uB5.1 (A->B)
- net at uC9.8 (Y3): now also uD5.1 (A->B)
- net at uC5.1 (A1): now also uF4.13 (Qh)
- net ~{CRTC-RA3}: now reaches uC5.10 (Y5)
- net ~{CRTC-RA3}: now also uE5.12 (H1)
- net at uC5.2 (Y1): now also uC4.2 (B1)
- net at uC5.3 (A2): now also uC4.3 (Y1)
- net at uC5.4 (Y2): now also uB4.6 (B2)
- net at uC5.5 (A3): now also uC4.8 (Y3), uC7.11 (K2)
- net at uC5.6 (Y3): now also uC7.8 (J2)
- net ~{CLK-2M}: now reaches uC5.8 (Y4)
- net ~{CLK-2M}: now also uE7.11 (Cp), uF6.20 (~{OE}), uF8.20 (~{OE})
- net ~{VRAM-WE}: now reaches uF8.21 (~{WE})
- net ~{VRAM-WE}: now also uD7.1 (OEa), uD7.19 (OEb), uF9.7 (Zb)
- net ~{CRAM-WE}: now reaches uF6.21 (~{WE})
- net ~{CRAM-WE}: now also uD4.1 (OEa), uD4.19 (OEb), uF7.7 (Zb)
- net FD-SEL1: now reaches J4.10 (Pin_10)
- net FD-SEL1: now also uC1.1 (Q0)
- net FD-SEL2: now reaches J4.12 (Pin_12)
- net FD-SEL2: now also uC1.2 (Q1)
- net FD-SEL3: now reaches J4.14 (Pin_14)
- net FD-SEL3: now also uC1.3 (Q2)
- net FD-HLD: now reaches J4.16 (Pin_16)
- net FD-HLD: now also uB1.8 (Y4)
- net FD-DIRC: now reaches J4.18 (Pin_18)
- net FD-DIRC: now also uB1.6 (Y3)
- net FD-STEP: now reaches J4.20 (Pin_20)
- net FD-STEP: now also uB1.10 (Y5)
- net FD-WRITE: now reaches J4.22 (Pin_22)
- net FD-WRITE: now also uB1.4 (Y2)
- net FD-WG: now reaches J4.24 (Pin_24)
- net FD-WG: now also uC0.3 (Y1)
- net FD-TRK0: now reaches J4.26 (Pin_26)
- net FD-TRK0: now also R7.2
- net FD-WP: now reaches J4.28 (Pin_28)
- net FD-WP: now also R8.2
- net FD-READ: now reaches J4.30 (Pin_30)
- net FD-READ: now also uD2.1 (A1)
- net FD-SIDE: now reaches J4.32 (Pin_32)
- net FD-SIDE: now also uB1.2 (Y1)
- net FD-RDY: now reaches J4.34 (Pin_34)
- net FD-RDY: now also uD2.13 (A6)
- net FD-SEL4: now reaches J4.6 (Pin_6)
- net FD-SEL4: now also uC1.4 (Q3)
- net FD-INDEX: now reaches J4.8 (Pin_8)
- net FD-INDEX: now also uD2.3 (A2)
- net at uC4.1 (A1): now also uB2.8 (~{Q2})
- net at uC4.10 (B3): now also uC7.3 (Q1)
- net CRTC-VS: now reaches uC4.4 (A2)
- net CRTC-VS: now also uC4.5 (B2), uD9.40 (VS)
- net ~{CRTC-VS}: now reaches uC4.6 (Y2)
- net ~{CRTC-VS}: now also uB4.2 (A1)
- net ~{VID-WE}: now reaches uF7.5 (I0b)
- net ~{VID-WE}: now also uF9.5 (I0b), uG4.12 (Y6)
- net at uF4.15 (PE): now also uE5.8 (Y1)
- net FDC-HLT: now reaches uE2.12 (~{Q2})
- net FDC-HLT: now also uD3.23 (HLT)
- net CRTC-DE: now reaches uE5.6 (F1)
- net CRTC-DE: now also uD9.18 (DE)
- net ~{FDC-INDEX}: now reaches uD2.10 (Y5)
- net ~{FDC-INDEX}: now also uD3.35 (~{IP})
- net FDC-INDEX: now reaches uD2.11 (A5)
- net FDC-INDEX: now also uD2.4 (Y2)
- net FDC-RDY: now reaches uD2.12 (Y6)
- net FDC-RDY: now also uD3.32 (READY)
- net ~{FD-READ}: now reaches uD2.2 (Y1)
- net ~{FD-READ}: now also uC2.2 (B1)
- net PPI-PC6: now reaches uF2.11 (PC6)
- net PPI-PC6: now also uB1.1 (A1)
- net PPI-PC5: now reaches uF2.12 (PC5)
- net PPI-PC5: now also uC1.14 (P1)
- net PPI-PC4: now reaches uF2.13 (PC4)
- net PPI-PC4: now also uC1.15 (P0)
- net PPI-PC3: now reaches uF2.17 (PC3)
- net PPI-PC3: now also C28.2
- net BUS-RST: now reaches uF2.35 (RESET)
- net BUS-RST: now also uF3.2 (Y1)
- net at uC7.13 (~{R1}): now also uC7.6 (~{Q2})
- net CLK-1M: now reaches uE4.11 (Q3)
- net CLK-1M: now also uD3.24 (CLK)
- net FDC-STEP: now reaches uD3.15 (STEP)
- net FDC-STEP: now also uB1.11 (A5)
- net FDC-DIRC: now reaches uD3.16 (DIRC)
- net ~{FDC-RAWRD}: now reaches uD3.27 (~{RAWRD})
- net ~{FDC-RAWRD}: now also uC2.4 (~{Q1})
- net FDC-HLD: now reaches uD3.28 (HLD)
- net FDC-HLD: now also uB1.9 (A4)
- net FDC-WG: now reaches uD3.30 (WG)
- net FDC-WG: now also uC0.1 (A1), uC0.2 (B1)
- net FDC-WRITE: now reaches uD3.31 (WD)
- net FDC-WRITE: now also uB1.3 (A2)
- net ~{FDC-TRK0}: now reaches uD3.34 (~{TRO0})
- net ~{FDC-TRK0}: now also R7.1
- net ~{FDC-WPRT}: now reaches uD3.36 (~{WPRT})
- net ~{FDC-WPRT}: now also R8.1
- net at BZ1.2 (-): now also Q1.2 (C)
- new net: D1.1 (K), Q1.3 (B)
- new net: C28.1, D1.2 (A)
- new net FDC-DRIC: uB1.5 (A3)
- no-connect marks 58 -> 76
Other:
- moved on the sheet: BZ1, C1, C10, C2, C20, C22, C3, C4, C5, C6, C7, C8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
