File: Mainboard/MBC-1000_Mainboard/MBC-1000_Mainboard.kicad_sch (KiCad schematic)
At the start: 128 parts, among them J1 Keyboard, J2 Conn_02x18_Counter_Clockwise, J3 Conn_01x08, J4 Conn_02x17_Odd_Even, J6 Conn_02x25_Odd_Even, J7 FG, Q1 D1111, U2 74LS32

Commit message: Mainboard video output logic
Parts:
- added J5: Conn_01x05, symbol Connector_Generic:Conn_01x05
- added R29: 330R, symbol Device:R_Small_US
- added R30, R46: 1k, symbol Device:R_Small_US
Connections:
- net GND: now also J5.3 (Pin_3)
- net VCC: now also R29.2, R30.2, R46.2
- net ~{CRTC-VS}: now also uB4.3 (B1)
- net VID-SHIFT: now reaches uC5.1 (A1), uF4.13 (Qh)
- net ~{VID-SHIFT}: now reaches uC4.2 (B1), uC5.2 (Y1)
- net VID-OUT_{1}: now reaches uC4.3 (Y1), uC5.3 (A2)
- net ~{VID-OUT}: now reaches uB4.6 (B2), uC5.4 (Y2)
- net ~{VID-OUT}: now also uB4.5 (A2)
- net ~{VID-HSYNC}: now reaches uC4.11 (Y4)
- net ~{VID-HSYNC}: now also uB4.11 (A4), uB4.12 (B4)
- net CRTC-HS: now reaches uC4.12 (A4)
- net CRTC-HS: now also uC4.13 (B4), uD9.39 (HS)
- net VID-VSYNC: now reaches uB4.1 (Y1)
- net VID-VSYNC: now also J5.5 (Pin_5), R30.1
- net VID-HSYNC: now reaches uB4.13 (Y4)
- net VID-HSYNC: now also J5.1 (Pin_1), R46.1
- net VID-OUT: now reaches uB4.4 (Y2)
- net VID-OUT: now also J5.4 (Pin_4), R29.1
- no-connect marks 76 -> 82

Commit message: Mainboard reversing continued
Parts:
- removed C1: C_Small, symbol Device:C_Small
- added C1: 470n, symbol Device:C_Polarized_Small_US
- added C12: 100n, symbol Device:C_Polarized_Small_US
- added C14: 0680J, symbol Device:C_Small
- added C25: 4700, symbol Device:C_Small
- added D2, D4, D5: D, symbol Device:D
- added R16: 8k2, symbol Device:R_Small_US
- added R17, R18: 9k1, symbol Device:R_Small_US
- added R19, R20, R21: 1M-1%, symbol Device:R_Small_US
- added R22, R31: 4k7, symbol Device:R_Small_US
- added R49: 100R, symbol Device:R_Small_US
- added R6: 560R, symbol Device:R_Small_US
Connections:
- net +12V: now also uA1.8 (V+)
- net GND: now also uA1.4 (V-), uA2.8 (GND), uC3.8 (GND), C25.2, R16.1, R21.2
- net VCC: now also uA2.10 (B2), uA2.11 (~{CLR2}), uA2.16 (VCC), uA2.3 (~{CLR1}), uB2.10 (~{S2}), uB2.4 (~{S1}), uC2.16 (VCC), uC2.3 (~{CLR1}), uC3.1 (~{MR}), uC3.10 (CET), uC3.16 (VCC), uC3.3 (D0), uC3.4 (D1), uC3.5 (D2), uC3.6 (D3), uC3.7 (CEP), uC3.9 (~{PE}), R20.2, R6.2
- net ~{CLK-2M}: now also uB2.11 (C2)
- net at uD1.2 (D1): now also uD2.6 (Y3)
- net at uC3.13 (Q1): now also uD3.26 (RCLK)
- net at uC3.14 (Q0): now also uA3.11 (3C), uB3.11 (A4), uF3.13 (A6)
- net at uC3.2 (CP): now also uA2.1 (~{A1}), uA2.5 (Q2)
- net at uB2.1 (~{R1}): now also uA2.2 (B1)
- net CRTC-CRSR: now reaches uB2.12 (D2)
- net at uB2.13 (~{R2}): now also R22.2
- net at uB2.2 (D1): now also uA3.9 (3A), uB3.12 (B4), uC2.5 (Q2)
- net at uB2.3 (C1): now also uF3.12 (Y6)
- net at uB2.5 (Q1): now also uA3.10 (3B), D2.1 (K)
- net at uD2.5 (A3): now also R49.2
- net at uA3.8 (3Y): now also R31.1
- net at uA2.13 (Q1): now also uA2.9 (~{A2})
- net at uA2.15 (RCext1): now also R17.2
- net at uA2.6 (Cext2): now also C14.1
- net at uA2.7 (RCext2): now also C14.2, R18.2
- net at uB3.13 (Y4): now also D4.1 (K)
- net at uA1.5 (I2+): now also C12.1, D5.2 (A), R20.1, R21.1
- net at uA1.6 (I2-): now also R19.2
- net at uA1.7 (O2): now also R17.1, R18.1, R19.1
- new net: C25.1, R49.1, R6.1
- new net: C12.2, R16.2
- new net: D2.2 (A), D4.2 (A), R22.1
- new net: D5.1 (K), R31.2
- no-connect marks 82 -> 104
Other:
- moved on the sheet: J5, R29, R30, R46

Commit message: Motherboard trace out final IC signals
Parts:
- added C15, C17: 2000J, symbol Device:C_Small
- added C23: 47u, symbol Device:C_Polarized_Small_US
- added C24, C29: 1nF, symbol Device:C_Small
- added C26, C27: 27, symbol Device:C_Small
- added JP2: Jumper_3_Bridged12, symbol Jumper:Jumper_3_Bridged12
- added R10, R48: 150R, symbol Device:R_Small_US
- added R11: 4k7-1%, symbol Device:R_Small_US
- added R14: 11k-1%, symbol Device:R_Small_US
- added R24, R5: 1k, symbol Device:R_Small_US
- added R9: 3k3, symbol Device:R_Small_US
- added RV1: R_Potentiometer_US, symbol Device:R_Potentiometer_US
- added VR1: 5k, symbol Device:R_Potentiometer_US
Connections:
- net BUS-RST: now also C24.1
- net CLK-16M: now also uF4.7 (Clk)
- net CLK-1M: now also uD1.3 (C1)
- net FD-RDY: now also R10.2
- net FD-READ: now also R48.2
- net FDC-HLD: now also uE2.10 (B2)
- net GND: now also uC2.8 (GND), uC2.9 (~{A2}), uE2.14 (Cext1), uE2.6 (Cext2), uE2.8 (GND), uE2.9 (A2), uF4.6 (CE), C23.2, C24.2, C26.2, C27.2, C29.2
- net LPT-ACK: now also JP2.1 (A), R9.2
- net LPT-BUSY: now also JP2.3 (B)
- net PPI-PC3: now also uD1.9 (Q2)
- net VCC: now also uC2.11 (~{CLR2}), uD1.1 (~{R1}), uD1.10 (~{S2}), uD1.12 (D2), uD1.4 (~{S1}), uE2.11 (Clr2), uE2.16 (VCC), R10.1, R11.2, R24.1, R48.1, R9.1, VR1.1, VR1.2
- net ~{CPU-RST}: now also C29.1
- net at uD1.11 (C2): now also uD1.5 (Q1), C27.1
- net PPI-PC7: now reaches uD1.13 (~{R2})
- net PPI-PC7: now also uE1.5 (A3), uF2.10 (PC7)
- net at uD1.2 (D1), uD2.6 (Y3): now also C26.1
- net at D1.1 (K), Q1.3 (B): now also C1.2
- net at uE2.7 (RCext2): now also C23.1
- net at uE1.6 (Y3): now also R24.2, R5.1
- net at C1.1: now also R5.2
- net PPI-PC2: now reaches uF2.16 (PC2)
- net PPI-PC2: now also uF3.6 (Y3)
- net at uC2.10 (B2): now also uC2.13 (Q1)
- net at uC2.14 (Cext1): now also C17.1
- net at uC2.15 (RCext1): now also C17.2, R11.1
- net at uC2.6 (Cext2): now also C15.2
- net at uC2.7 (RCext2): now also C15.1, R14.2
- net at uF3.3 (A2): now also JP2.2 (C)
- net at uF3.4 (Y2): now also uF3.5 (A3)
- new net: R14.1, VR1.3
- no-connect marks 104 -> 130
Other:
- moved on the sheet: BZ1, C1, C28, D1, JP1, Q1
